File: LM2596project.kicad_pcb (KiCad board)
At the start: 2 copper layers, 56.8 x 32.8 mm, 17 parts, among them J1 Screw_Terminal_01x02, J2 Screw_Terminal_01x02, U1 LM2596S-ADJ

Commit message: Add files via upload
Parts:
- removed the G*** at (36.7, 122.8)
